File: elec/usb2ax_pro_main_v1.0.brd (EAGLE design)
At the start: 44 x 32 mm, 64 parts, among them J1 MICRO-USB-5P-340015001, J3 M10X2_SMD_1.27_FEMALE, K1 BUTTON-2P-REINFORCE-3100060P1, P1 PIN_SMD_2X2.5, P10 PIN_SMD_0.8X1.6, P11 PIN_SMD_0.8X1.6, P12 PIN_SMD_0.8X1.6, P13 PIN_SMD_1X2, P14 PIN_SMD_0.8X1.6, P15 PIN_SMD_0.8X1.6, P16 PIN_SMD_1X2, P2 PIN_SMD_2X2.5, P3 PIN_SMD_0.8X1.6, P4 PIN_SMD_0.8X1.6, P5 PIN_SMD_1X2, P6 PIN_SMD_1X2, P7 PIN_SMD_1X2, P8 PIN_SMD_1X2, P9 PIN_SMD_1X2, U1 ATSAM3U_C-AU, U2 MIC5205-3.3YM5, U3 BR24G256FJ-3AGTE2, U6 MPU-6050, X1 12MHz

Commit message: Fixed 3V3 reg value
Parts:
- U2: value MIC5205-3.3YM5 -> NCP5025Q33T2G
Changed lines of the file:
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@@
 <element name="X1" library="OPL" package="2P-SMD-5.0X3.2" value="12MHz" x="5.35" y="15.1" rot="R270"/>
 <element name="C12" library="Xevelabs" package="0805_N" value="10uF" x="29.65" y="18.35"/>
-<element name="U2" library="OPL" package="SC70-5" value="MIC5205-3.3YM5" x="29.1" y="15.9"/>
+<element name="U2" library="OPL" package="SC70-5" value="NCP5025Q33T2G" x="29.1" y="15.9"/>
 <element name="C13" library="Xevelabs" package="0201_N" value="470pF" x="31" y="15.9" rot="R270"/>
 <element name="C1" library="Xevelabs" package="0201_N" value="0.1uF" x="26.7" y="20.1" rot="R90"/>
